File: hardware/Blinkenstar/Blinkenstar.kicad_pcb (KiCad board)
At the start: 2 copper layers, 84.4 x 82.8 mm, 22 parts, among them J1 AudioJack2_Ground, J3 CLKI, U2 ATtiny88-A, U3 EEPROM-I2CEIAJ

Commit message: Update Blinkenstar configuration and production files
- Added "OPEN BROWSER" and "NO_BACKUP_OPT" options to fabrication-toolkit-options.json.
- Introduced new production zip file Blinkenstar_2.9.zip.
- Created backup zip file Blinkenstar_2.9_2026-05-14_22-12-31.zip.
- Modified netlist.ipc to update VIA connections, replacing several with new identifiers and removing obsolete entries.
- Adjusted J1 connections in netlist.ipc for improved clarity and accuracy.
Other:
- board text added: "v2.9"
- board text removed: "v2.8"
